File: 780nm-ecdl-grating/780nm-ecdl-grating.kicad_sch (KiCad schematic)
At the start: 78 parts, among them IC1 OPA192IDR, IC2 OPA192IDR, IC3 OPA192IDR, IC4 OPA462IDDAR, IC5 OPA192IDR, J1 RP INPUT, J2 1755736, J3 TSW-103-07-G-S, J4 1755736, J5 MON OUT, U1 ADR4550, U2 BAV199Q-7-F

Commit message: added analog supply sec
Parts:
- added C31, C35: 4.7u, symbol Device:C
- added C32, C34, C36, C37: 0.1u, symbol Device:C
- added C33, C38: 10n, symbol Device:C
- added FB1, FB2: 1000 ohms, symbol Device:FerriteBead
- added TP5: V_MON, symbol Connector:TestPoint
Connections:
- net +9V: now also C33.1, C34.1, FB1.2
- net -5V: now also C37.1, C38.1, FB2.2
- net GND: now also C31.2, C32.2, C33.2, C34.2, C35.2, C36.2, C37.2, C38.2; no longer R17.2
- net V_MON: now also TP5.1
- new net +3.3V: R17.2
- new net +9V_IN: C31.1, C32.1, FB1.1
- new net -5V_IN: C35.1, C36.1, FB2.1
Other:
- note added: "Input Power Supply"

Commit message: power correction for OPA462
Parts:
- added C39, C40: 22u, symbol Device:C
Connections:
- net +9V_IN: now also C39.1
- net -5V: no longer D1.2 (A), D4.2 (A2), IC4.4 (V-), IC4.9 (EP)
- net -5V_IN: now also D1.2 (A), D4.2 (A2), IC4.4 (V-), IC4.9 (EP), C40.1
- net GND: now also C39.2, C40.2
Other:
- moved on the sheet: C31, C32, C33, C34, C35, C36, C37, C38, FB1, FB2

Commit message: forgot to add DPDT and status
Parts:
- added D6, D7: LED, symbol Device:LED
- added J6: 1715734, 1715734, symbol 1715734:1715734
- added R22: 3.3k, Resistor_SMD:R_1206_3216Metric, symbol Device:R
- added R24: 1.2k, Resistor_SMD:R_1206_3216Metric, symbol Device:R
- added S1: B22AP, B22AP, symbol B22AP:B22AP
Connections:
- net +9V_IN: now also R22.1, S1.2 (COM_1)
- net -5V_IN: now also R24.1, S1.5 (COM_2)
- net GND: now also D6.1 (K), D7.2 (A), J6.2
- new net: D7.1 (K), R24.2
- new net: D6.2 (A), R22.2
- new net +9V_SW: J6.1, S1.1 (NO_1)
- new net -5V_SW: J6.3, S1.4 (NO_2)
- no-connect marks 12 -> 14
Other:
- note added: "DPDT PWR switch"
- note added: "PWR Status LEDs"
- note added: "PWR term blk."

Commit message: finally done!
Parts:
- added C41, C42: 4.7u, symbol Device:C
Connections:
- net +9V: now also C41.1
- net +9V_IN: no longer R22.1
- net +9V_SW: now also R22.1
- net -5V: now also C42.1
- net -5V_IN: no longer R24.1
- net -5V_SW: now also R24.1
- net GND: now also C41.2, C42.2
Other:
- moved on the sheet: FB1, FB2

Commit message: assigned footprints
Parts:
- C1, C11, C12, C13, C15, C16, C17, C2, C21, C22, C26, C27, C3, C30, C31, C32, C34, C35, C36, C37, C41, C42, C5, C6, C8, C9: footprint (none) -> Capacitor_SMD:C_0603_1608Metric
- C10, C18, C19, C29, C33, C38, C7, R4: footprint (none) -> Capacitor_SMD:C_0402_1005Metric
- C14, C39, C4, C40: footprint (none) -> Capacitor_SMD:C_0805_2012Metric
- C20, R16, R17, R2, R29, R3, R5, R6, R7, R8, R9: footprint (none) -> Resistor_SMD:R_0603_1608Metric
- C23: value 10u -> 22u; footprint (none) -> UCS2E220MPD:PCAP_10x20-THRU-ELECT_NCA
- C24: footprint (none) -> ECA-2EHG100B:CAP_PAN_10X16_PAN
- C25: footprint (none) -> PHE426HA6100JR05:CAP_PHE426_AH_KEM
- C28: footprint (none) -> Capacitor_SMD:C_1206_3216Metric
- CR1: footprint DFN1006-2_SOD882_NEX -> PESD5V0V1BL:DFN1006-2_SOD882_NEX
- D6, D7: footprint (none) -> LED_SMD:LED_0603_1608Metric
- FB1, FB2: footprint (none) -> Inductor_SMD:L_0603_1608Metric
- IC1, IC2, IC3, IC5: footprint SOIC127P600X175-8N -> OPA192:SOIC127P600X175-8N
- IC4: footprint SOIC127P600X170-9N -> OPA462:SOIC127P600X170-9N
- J1: footprint (none) -> SMA-J-P-H-ST-TH1:CONN_SMA-J-P-H-ST-TH1_SAI
- J2, J4: footprint 1755736 -> 1755736:1755736
- J3: footprint TSW-103-XX-YY-S -> TSW-103-07-G-S:TSW-103-XX-YY-S
- J5: footprint (none) -> 731000105:CONN_73100-0105_MOL
- J6: footprint 1715734 -> 1715734:1715734
- R1: footprint POT_3296W -> 3296W-1-103LF:POT_3296W
- R10, R11: footprint (none) -> Resistor_SMD:R_0402_1005Metric
- R12, R13, R28: footprint (none) -> Resistor_SMD:R_1206_3216Metric
- R14, R15: footprint (none) -> Resistor_SMD:R_1210_3225Metric
- R22, R24: footprint Resistor_SMD:R_1206_3216Metric -> Resistor_SMD:R_0603_1608Metric
- RN1: footprint ACASA1002S1002P100:RESCAXS80P320X150X55-8N -> ACASA1002:RESCAXS80P320X150X55-8N
- S1: footprint B22AP -> B22AP:B22AP
- TP1, TP2, TP3, TP4, TP5: footprint (none) -> TestPoint:TestPoint_Keystone_5015_Micro_Mini
- U2: footprint SOT23_BAV_DIO -> BAV199Q-7-F:SOT23_BAV_DIO
Other:
- note added: "+155V output"

Commit message: almost done with layout
Parts:
- removed J6: 1715734, 1715734:1715734, symbol 1715734:1715734
- added C43: 10u, Capacitor_SMD:C_0603_1608Metric, symbol Device:C
- added C44: 0.1u, Capacitor_SMD:C_0603_1608Metric, symbol Device:C
- added C45: 10n, Capacitor_SMD:C_0402_1005Metric, symbol Device:C
- added D8: LED, LED_SMD:LED_0603_1608Metric, symbol Device:LED
- added J7: 1715747, 1715747:1715747, symbol 1715747:1715747
- added R25, R26: 1k, Resistor_SMD:R_0603_1608Metric, symbol Device:R
- added TP6, TP7: TestPoint, TestPoint:TestPoint_Pad_D4.0mm, symbol Connector:TestPoint
- C23, C24: symbol Device:C -> Device:C_Polarized
- CR1: footprint PESD5V0V1BL:DFN1006-2_SOD882_NEX -> PESD5V0F1BL:DFN1006-2_SOD882_NEX
- J5: footprint 731000105:CONN_73100-0105_MOL -> 112404:CONN_112404_AMP
Connections:
- net +155V: now also TP7.1
- net +9V_SW: now also J7.1
- net -5V: no longer C21.2, C22.2
- net -5V_IN: now also C21.2, C22.2, C43.2
- net -5V_SW: now also J7.4
- net E/D: now also R26.1; no longer J3.1
- net GND: now also C43.1, C44.2, C45.2, D8.1 (K), J7.3
- net at C20.2, D1.1 (K), D2.2 (A)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: now also TP6.1
- net +3.3V renamed +3.3V_SW
- net +3.3V_SW: now also C44.1, C45.1, J7.2, R25.1
- new net: J3.1, R26.2
- new net: D8.2 (A), R25.2
Other:
- note added: "3.3V rail"
- moved on the sheet: C21, C22, D6, D7, R13, R22, R24, S1
