File: 780nm-ecdl-grating/780nm-ecdl-grating.kicad_pcb (KiCad board)
At the start: 2 copper layers, 94.9 x 56.4 mm, 112 parts, among them IC1 OPA192IDR, IC2 OPA192IDR, IC3 OPA192IDR, IC4 OPA462IDDAR, IC5 OPA192IDR, J1 RP INPUT, J2 1755736, J3 TSW-103-07-G-S, J4 1755736, J5 MON OUT, J7 1715747, U1 ADR4550, U2 BAV199Q-7-F

Commit message: finished layout
Parts:
- added REF**: Symbol_HighVoltage_Triangle_6x6mm_Copper, Symbol:Symbol_HighVoltage_Triangle_6x6mm_Copper, F.Cu at (227.6, 66.8)
- added REF**: Symbol_HighVoltage_Triangle_6x6mm_Copper, Symbol:Symbol_HighVoltage_Triangle_6x6mm_Copper, F.Cu at (224.0, 43.9)
- HV RAW: renamed from TP6
- HV TEST: renamed from TP7
- SUM OUT: renamed from TP4
- moved R18 185.5 mm to (241.6, 73.0), turned to -90 degrees
- moved R19 184.1 mm to (240.1, 77.0), turned to 180 degrees
- moved C24 168.6 mm to (246.5, 71.5)
- moved R13 167.3 mm to (223.4, 65.6), turned to 90 degrees
- moved R20 165.8 mm to (221.9, 69.6), turned to 180 degrees
- moved R28 162.0 mm to (217.9, 77.0), turned to -90 degrees
- moved R23 161.0 mm to (216.9, 69.6), turned to 180 degrees
- moved R27 157.0 mm to (212.8, 70.7), turned to -90 degrees
- moved IC5 154.5 mm to (210.2, 78.7), turned to -90 degrees
- moved R21 153.9 mm to (210.0, 70.7), turned to 90 degrees
- moved C23 153.8 mm to (246.0, 83.4)
- moved R12 152.8 mm to (208.7, 48.3), turned to 90 degrees
- moved J4 151.8 mm to (228.7, 92.0)
- moved C29 145.9 mm to (211.3, 84.7), turned to 90 degrees
- moved C27 144.7 mm to (221.1, 71.8), turned to 180 degrees
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Connections:
- J5 pad 3: (no net) -> GND
- J5 pad 4: (no net) -> GND
- J5 pad 5: (no net) -> GND
Other:
- board size 94.9 x 56.4 mm -> 112.6 x 58.3 mm
- board text added: "+155V"
- board text added: "DANGER HIGH VOLTAGE"
- board text added: "PIEZO"

Commit message: added safety measures
Parts:
- added SYM: Caution_Hot_Surface_FinalFit_12x12mm_Silk, CAUTION_HOT:Caution_Hot_Surface_FinalFit_12x12mm_Silk, F.Cu at (154.1, 74.8)
- added SYM: Caution_Hot_Surface_FinalFit_12x12mm_Silk, CAUTION_HOT:Caution_Hot_Surface_FinalFit_12x12mm_Silk, F.Cu at (203.7, 64.5)
- moved D4 1.07 mm to (210.2, 60.7)
- moved C43 1.07 mm to (207.0, 58.7)

Commit message: completed layout v0
Parts:
- removed the SYM at (154.1, 74.8)
- HV MONITOR: renamed from TP5
- moved SUM OUT 5.18 mm to (201.3, 55.9)
- moved HV MONITOR 0.87 mm to (203.7, 85.1), turned to 90 degrees
- moved TP1 0.78 mm to (184.8, 59.0)
- moved R2 0.70 mm to (160.4, 63.7)
- moved C28 0.63 mm to (205.6, 72.5)
- moved R27 0.55 mm to (212.3, 71.0)
- moved R21 0.53 mm to (209.6, 71.0)
- moved C4 0.38 mm to (170.1, 64.9)
- moved R1 0.38 mm to (164.4, 64.6)
- moved R3 0.32 mm to (169.2, 62.0)
- moved C14 0.28 mm to (180.7, 64.8)
- moved R6 0.28 mm to (175.3, 65.3)
- moved C7 0.27 mm to (174.4, 57.8)
- moved IC1 0.27 mm to (175.3, 61.4)
- moved R4 0.27 mm to (170.8, 59.5)
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Routing:
- net E/D: track 0.00 -> 72.9 mm, vias 0 -> 2
- net PIEZO_OUT: track 0.00 -> 68.0 mm
- net STATUS: track 0.00 -> 67.0 mm, vias 0 -> 2
- net Net-(D1-K): track 0.00 -> 36.3 mm
- net SUM_OUT: track 0.00 -> 35.5 mm
- net +3.3V_SW: track 0.00 -> 33.6 mm, vias 0 -> 2
- net +155V: track 0.00 -> 31.3 mm, vias 0 -> 4
- net +9V: track 0.00 -> 28.5 mm, vias 0 -> 6
- net V_MON: track 0.00 -> 26.6 mm
- net CMD_IN: track 0.00 -> 25.1 mm
- net RP_BUFF_OUT: track 0.00 -> 23.9 mm
- net Net-(D7-K): track 0.00 -> 21.2 mm
- net REF_BUFF_OUT: track 0.00 -> 18.8 mm
- net Net-(D8-A): track 0.00 -> 17.6 mm
- net Net-(IC5-+IN): track 0.00 -> 17.5 mm
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- added copper zone on In2.Cu, net +155V
- added copper zone on In2.Cu, net +3.3V_SW
- added copper zone on B.Cu, net +9V
- added copper zone on F.Cu, net +9V
- added copper zone on In2.Cu, net +9V
- added copper zone on F.Cu, net +9V_IN
- added copper zone on In2.Cu, net +9V_IN
- added copper zone on B.Cu, net +9V_SW
- added copper zone on In2.Cu, net +9V_SW
- added copper zone on F.Cu, net -5V
- added copper zone on In2.Cu, net -5V
- added copper zone on B.Cu, net -5V_IN
- added copper zone on F.Cu, net -5V_IN
- added copper zone on In2.Cu, net -5V_IN
- added copper zone on B.Cu, net -5V_SW
- added copper zone on In2.Cu, net -5V_SW
- added copper zone on B.Cu, net GND
- added copper zone on F.Cu, net GND
- added copper zone on In1.Cu, net GND
- added copper zone on In2.Cu, net GND
Other:
- copper layers 2 -> 4
- board text added: "REFERENCE BIAS"

Commit message: completed DRC
Routing:
- net RP_IN: track 8.57 -> 15.6 mm
- net GND: track 0.00 -> 6.19 mm, vias 0 -> 8
- net +9V: track 28.5 -> 31.4 mm, vias 6 -> 9
- net +155V: track 31.3 -> 33.6 mm, vias 4 -> 5
- net SUM_OUT: track 35.5 -> 36.3 mm
- net -5V_IN: vias 22 -> 21
- net +9V_IN: vias 0 -> 3
Other:
- board text added: "MONITOR HV"
- board text added: "PIEZO OUTPUT"
- board text added: "SHUTDOWN: E/D LOW → RP DAC = 0 V → ±LV OFF → +155 V OFF"
- board text added: "STARTUP: E/D LOW → RP DAC = 0 V → +155 V ON → ±LV ON → WAIT 0.5-1 s → E/D HIGH"
