File: ecdl-laser-bboard/sch3.kicad_sch (KiCad schematic)
At the start: 14 parts, among them IC4 OPA4192IPWR, J10 SET T MON, J11 SET T MON, J8 LD I MON, J9 LD P MON

Commit message: begun layout
Parts:
- added J12: TSS-106-01-L-D, TSS-106-01-L-D:TSS-106-XX-YYY-D, symbol TSS-106-01-L-D:TSS-106-01-L-D
- added TP11: EXT T SET, TestPoint:TestPoint_Keystone_5015_Micro_Mini, symbol Connector:TestPoint
- IC4: footprint SOP65P640X120-14N -> OPA4192:SOP65P640X120-14N
- J10, J11, J8, J9: footprint (none) -> 112404:CONN_112404_AMP
- R77, R78, R79, R80, R81: footprint (none) -> Resistor_SMD:R_0603_1608Metric
Connections:
- net EXT_T_SET: now also TP11.1
- net LDTC_COM: now also J12.11, J12.3, J12.7
- net V_NEG: now also C69.1, C70.1, IC4.11 (V-)
- new net +3.3VRP: J12.1
- new net AIN0: J12.8
- new net AIN1: J12.6
- new net AIN2: J12.4
- new net AIN3: J12.2
- new net DAC_SCLK: J12.9
- new net DAC_SDIN: J12.5
- new net DAC_SYNC: J12.12
- new net RP_EN: J12.10
Other:
- note added: "(Pololu 4584)"
- note added: "Monitor BNC's"
- note added: "Monitor Buffers"
- note added: "RP Connections"
- note added: "Temp Set"

Commit message: pre-chipotle layout
Changed lines of the file:
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@@
+		)
+	)
+	(polyline
+		(pts
+			(xy 92.075 149.86) (xy 64.77 149.86)
+		)
+		(stroke
+			(width 0)
+			(type default)
 		)
 	)

Commit message: layout complete!
Connections:
- net LD_P_MON_out: no longer IC4.8 (OUT_C)
- new net SET_T_MON_out: IC4.8 (OUT_C)
Changed lines of the file:
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@@
 		)
 	)
-	(global_label "LD_P_MON_out"
+	(global_label "SET_T_MON_out"
 		(shape input)
 		(at 82.55 39.37 270)
@@
 		)
 		(property "Intersheetrefs" "${INTERSHEET_REFS}"
-			(at 82.55 55.9622 90)
+			(at 82.55 56.6878 90)
 			(hide yes)
 			(show_name no)
