File: ecdl-laser-bboard/ecdl-laser-bboard.kicad_pcb (KiCad board)
At the start: 2 copper layers, 195 parts, among them IC1 DAC80501ZDGSR, IC2 OPA4192IPWR, IC3 LM7705MM_NOPB, IC4 OPA4192IPWR, J1 TEC control, J10 SET T MON, J11 SET T MON, J12 TSS-106-01-L-D, J13 M20-9980346, J2 Laser Control, J3 54-00166, J4 J_LDTC_LOAD, J5 J_LDTC_PWR, J6 J_LDTC_IO, J7 Conn_Coaxial, J8 LD I MON, J9 LD P MON, Q1 2N7002, U1 LT8624SAV-PBF, U2 LT8624SAV-PBF, U3 TPS259474LRPWR

Commit message: layout v0
Parts:
- added G***: LOGO, posm-logo:posm-logo-footprint, F.Cu at (125.1, 132.1)
- added REF**: MountingHole_3.2mm_M3, MountingHole:MountingHole_3.2mm_M3, F.Cu at (261.2, 135.1)
- added REF**: MountingHole_3.2mm_M3, MountingHole:MountingHole_3.2mm_M3, F.Cu at (104.7, 37.7)
- added REF**: MountingHole_3.2mm_M3, MountingHole:MountingHole_3.2mm_M3, F.Cu at (261.2, 37.9)
- added REF**: MountingHole_3.2mm_M3, MountingHole:MountingHole_3.2mm_M3, F.Cu at (104.8, 134.9)
- C6: footprint Capacitor_SMD:C_0603_1608Metric -> Capacitor_SMD:C_1210_3225Metric
- R30: value 7.5k -> 63.4k
- R35, R36, R37: value 33 -> 1k
- moved J2 211.9 mm to (233.3, 44.7)
- moved J4 194.4 mm to (213.1, 45.6), turned to 180 degrees
- moved J6 179.8 mm to (184.3, 128.7)
- moved J12 165.5 mm to (250.7, 130.9), turned to 180 degrees
- moved C20 108.8 mm to (131.8, 124.0), turned to 180 degrees
- moved J1 105.8 mm to (140.3, 43.1), turned to 180 degrees
- moved C22 103.1 mm to (159.1, 119.6)
- moved C23 102.9 mm to (159.1, 123.3)
- moved R18 102.3 mm to (136.2, 121.2), turned to -90 degrees
- moved C24 101.6 mm to (157.6, 127.8), turned to -90 degrees
- moved C38 100.4 mm to (-6.38, 50.9)
- moved C39 100.4 mm to (-6.38, 53.4)
- moved C40 100.4 mm to (-6.38, 55.9)
- moved C41 100.4 mm to (-6.38, 58.4)
- moved C42 100.4 mm to (-6.38, 60.9)
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- renumbered TP2 to +5V
Connections:
- IC2 pad 13: LDTC_COM -> Net-(IC2--_IN_D)
- IC2 pad 14: LDTC_COM -> Net-(IC2--_IN_D)
Other:
- board outline added: 165.4 x 105.7 mm
- board text added: "+12V INPUT"
- board text added: "+5V"
- board text added: "+V_FL"
- board text added: "+V_TEC"
- board text added: "+V_WTC"
- board text added: "Analog Rail"
- board text added: "J1 LDTC (PWR)"
- board text added: "TEC Rail"
- board text added: "V_FL"
- board text added: "V_WTC/V_TEC"
- board text added: "ecdl-laser controller board v0"

Commit message: pre-chipotle layout
Parts:
- added LDTC-COM: 5019, 5019:5019, F.Cu at (247.4, 100.1)
- added LDTC-COM: 5019, 5019:5019, F.Cu at (247.4, 72.0)
- added LDTC-COM: 5019, 5019:5019, F.Cu at (247.4, 85.5)
- added LDTC-COM: 5019, 5019:5019, F.Cu at (247.4, 58.1)
- BUFF BIAS: renamed from TP7
- BUFF MOD: renamed from TP5
- CURRENT MOD TP: renamed from TP6
- J2 LDTC (CONTROL): renamed from J6
- LD EN: renamed from TP10
- moved J11 266.3 mm to (256.1, 106.6)
- moved J10 266.0 mm to (256.1, 92.5)
- moved J9 265.6 mm to (256.1, 78.4)
- moved J8 265.3 mm to (256.1, 64.4)
- moved R29 256.3 mm to (246.9, 135.7), turned to -90 degrees
- moved R81 256.2 mm to (247.8, 106.6), turned to 180 degrees
- moved R28 255.5 mm to (246.1, 133.0)
- moved R80 252.5 mm to (247.9, 92.5), turned to 180 degrees
- moved R79 249.2 mm to (247.9, 78.4), turned to 180 degrees
- moved R78 246.4 mm to (247.8, 64.4), turned to 180 degrees
- moved LD EN 244.1 mm to (255.6, 131.7), turned to -90 degrees
- moved Q1 243.3 mm to (250.0, 132.1), turned to 90 degrees
- moved D5 237.2 mm to (251.6, 136.3)
- moved R1 234.7 mm to (220.6, 40.0), turned to 180 degrees
- moved C45 222.6 mm to (215.4, 87.3), turned to -90 degrees
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Connections:
- J2 pad 10: (no net) -> CHASSIS
- J2 pad 11: (no net) -> CHASSIS
- J7 pad 3: (no net) -> LDTC_COM
- J7 pad 4: (no net) -> LDTC_COM
- J7 pad 5: (no net) -> LDTC_COM
- J8 pad 3: (no net) -> LDTC_COM
- J8 pad 4: (no net) -> LDTC_COM
- J8 pad 5: (no net) -> LDTC_COM
- J9 pad 3: (no net) -> LDTC_COM
- J9 pad 4: (no net) -> LDTC_COM
- J9 pad 5: (no net) -> LDTC_COM
Routing:
- net LDA: track 0.00 -> 50.4 mm
- net LDC: track 0.00 -> 43.5 mm
- net PDA: track 0.00 -> 33.7 mm
- net SEN_P: track 0.00 -> 33.3 mm
- net SEN_N: track 0.00 -> 25.1 mm
- net Net-(J2-Pad6): track 0.00 -> 14.0 mm
- added copper zone on In2.Cu, net TEC_N
- added copper zone on In2.Cu, net TEC_P
Other:
- copper layers 2 -> 4
- board text added: "-0.23 V @ 25C"
- board text added: "224B LASER CONNECTOR"
- board text added: "224B TEC CONNECTOR"
- board text added: "ACT T MON"
- board text added: "CURRENT BIAS (0-1.25 V)"
- board text added: "CURRENT MOD SELECT"
- board text added: "DAC SPI"
- board text added: "HIGH --> 5 mA/V"
- board text added: "J3 LDTC (LD, PD, TEC)"
- board text added: "LD EN"
- board text added: "LD I MON"
- board text added: "LD P MON"
- board text added: "LOW --> 0.16 mA/V"
- board text added: "MED --> 1.61 mA/V"
- board text added: "NEGATIVE REF VOLTAGE"
- board text added: "RP DAC FAST"
- board text added: "SET T MON"
- board text added: "±2 V, Hi-Z"

Commit message: layout complete!
Parts:
- BUFF SUM: renamed from TP8
- C52 : renamed from C52
- EXT LD SET: renamed from TP9
- EXT T TEST: renamed from TP11
- LDTC COM: renamed from LDTC-COM (x4)
- moved R24 271.1 mm to (257.7, 43.3)
- moved R58 247.2 mm to (245.3, 130.8), turned to 180 degrees
- moved C70 244.5 mm to (231.4, 103.5)
- moved R64 242.4 mm to (245.3, 127.7), turned to 180 degrees
- moved C69 241.6 mm to (230.7, 95.3), turned to -90 degrees
- moved R70 240.9 mm to (245.3, 124.7), turned to 180 degrees
- moved R77 239.7 mm to (222.4, 114.1), turned to -90 degrees
- moved C56 239.3 mm to (235.8, 86.4), turned to -90 degrees
- moved C67 239.3 mm to (235.9, 92.4), turned to 90 degrees
- moved C58 238.1 mm to (230.7, 83.3), turned to 90 degrees
- moved C57 236.9 mm to (231.4, 75.3)
- moved R76 235.4 mm to (244.5, 119.6), turned to -90 degrees
- moved C59 235.4 mm to (244.9, 129.4)
- moved C62 233.1 mm to (244.9, 126.3)
- moved C65 231.1 mm to (244.9, 123.2)
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- renumbered TP3 to +12V, TP1 to +5V
Connections:
- IC4 pad 8: LD_P_MON_out -> SET_T_MON_out
Other:
- board text added: "(DNP)"
- board text added: "DNP"
- board text added: "EXT LD SET"
- board text added: "EXT T SET"
- board text added: "GND"
- board text added: "LDTC COM"
- board text added: "LP P MON"
- board text added: "NC"
- board text added: "OUTPUT MONITOR BUFFER"
- board text added: "RP GPIO"

Commit message: finalized layout v1
Parts:
- moved R25 124.9 mm to (170.1, 135.1), turned to 0 degrees
- moved C70 8.27 mm to (232.3, 95.3), turned to -90 degrees
- moved C57 8.07 mm to (232.4, 83.3), turned to 90 degrees
- moved EXT LD SET 7.09 mm to (187.0, 110.3)
- moved BUFF BIAS 6.62 mm to (200.3, 91.5)
- moved R75 5.95 mm to (238.2, 95.5), turned to 90 degrees
- moved C52  3.24 mm to (200.3, 112.8)
- moved R56 1.81 mm to (235.2, 83.4)
- moved R57 1.81 mm to (234.4, 80.8)
- moved R71 1.03 mm to (234.3, 95.5), turned to 90 degrees
- moved R55 0.74 mm to (236.2, 80.8), turned to 90 degrees
- moved EXT T TEST 0.46 mm to (226.3, 114.9)
- moved R6 0.16 mm to (134.2, 102.2)
- moved R17 0.14 mm to (134.3, 121.2)
- moved C51 0.07 mm to (199.4, 98.3)
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Connections:
- J3 pad A: (no net) -> +12V_RAW1
- J3 pad C: (no net) -> GND
- R24 pad 2: GND -> LDTC_COM
Routing:
- net DAC_SYNC: track 0.00 -> 119.8 mm, vias 0 -> 2
- net V_LDI_MON_OUT: track 0.00 -> 106.0 mm, vias 0 -> 2
- net DAC_SDIN: track 0.00 -> 102.8 mm, vias 0 -> 1
- net DAC_SCLK: track 0.00 -> 95.5 mm, vias 0 -> 2
- net +3.3VRP: track 0.00 -> 91.2 mm, vias 0 -> 1
- net +5V: track 0.00 -> 89.7 mm, vias 0 -> 44
- net V_LDP_MON_OUT: track 0.00 -> 82.3 mm, vias 0 -> 3
- net LD_SHD: track 0.00 -> 76.5 mm, vias 0 -> 1
- net V_SET_T_MON_OUT: track 0.00 -> 71.6 mm, vias 0 -> 3
- net V_FL: track 0.00 -> 68.9 mm, vias 0 -> 44
- net V_FINE_RAW: track 0.00 -> 53.1 mm
- net V_ACT_T_MON_OUT: track 0.00 -> 42.6 mm
- net LD_P_MON_+: track 0.00 -> 39.9 mm, vias 0 -> 2
- net LD_I_MON_+: track 0.00 -> 39.7 mm, vias 0 -> 2
- net ACT_T_MON_+: track 0.00 -> 34.5 mm, vias 0 -> 2
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- added copper zone on F.Cu, net +12V
- added copper zone on In2.Cu, net +12V
- added copper zone on F.Cu, net +12V_RAW1
- added copper zone on F.Cu, net +12V_RAW2
- added copper zone on In2.Cu, net +12V_RAW2
- added copper zone on F.Cu, net +5V
- added copper zone on In2.Cu, net +5V
- added copper zone on F.Cu, net +5V1
- added copper zone on F.Cu, net +5V2
- added copper zone on F.Cu, net CHASSIS
- added copper zone on In2.Cu, net CHASSIS
- added copper zone on B.Cu, net GND
- added copper zone on F.Cu, net GND
- added copper zone on In1.Cu, net GND
- added copper zone on In2.Cu, net GND
- added copper zone on B.Cu, net LDTC_COM
- added copper zone on F.Cu, net LDTC_COM
- added copper zone on In1.Cu, net LDTC_COM
- added copper zone on In2.Cu, net LDTC_COM
- added copper zone on F.Cu, net Net-(F1-Pad2)
- added copper zone on F.Cu, net Net-(J5-Pad2)
- added copper zone on F.Cu, net Net-(J5-Pad3)
- added copper zone on F.Cu, net SW
- added copper zone on F.Cu, net SW1
- added copper zone on B.Cu, net V_FL
- added copper zone on F.Cu, net V_FL
- added copper zone on In2.Cu, net V_FL
- added copper zone on F.Cu, net V_NEG
- added copper zone on In2.Cu, net V_NEG
Other:
- board text added: "ANALOG RAIL"
- board text added: "GROUND SPLIT JUMPER"
- board text added: "TEC RAIL"
- board text removed: "Analog Rail"
- board text removed: "TEC Rail"

Commit message: done?
Other:
- board text removed: "DNP"

Commit message: fixed bb board
Routing:
- net LDTC_COM: track 7.33 -> 8.15 mm, vias 563 -> 564
Changed lines of the file:
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@@
+	)
+	(segment
+		(start 172.543941 65.45)
+		(end 172.543941 65.473941)
+		(width 0.2)
+		(layer "F.Cu")
+		(net "LDTC_COM")
 	)
 	(segment
@@
 	)
 	(segment
+		(start 172.56 65.46)
+		(end 172.56 66.26)
+		(width 0.2)
+		(layer "F.Cu")
+		(net "LDTC_COM")
+	)
+	(segment
 		(start 200.175 98.28)
 		(end 201.09 98.28)
@@
 		(size 0.6)
 		(drill 0.3)
+		(layers "F.Cu" "B.Cu")
+		(free yes)
+		(net "LDTC_COM")
+	)
+	(via
+		(at 172.59 66.57)
+		(size 0.6)
+		(drill 0.3)
